File: Main.kicad_sch (KiCad schematic)
At the start: 446 parts, among them J1 Conn_02x22_Top_Bottom, Q1 2SC1384, Q2 2SC1384, SW1 SW_DIP_x08, U1 Conn_02x08_Counter_Clockwise, U10 7416, U100 74LS153, U101 74LS86, U102 74LS151, U103 74LS153, U104 74LS279, U105 74LS00, U106 74LS08, U107 NE555P, U108 74LS161, U109 74LS107, U11 7416, U110 74LS10, U111 74LS157, U112 74LS161, U113 74LS161, U114 74LS107, U115 Conn_02x08_Counter_Clockwise, U116 74LS175, U117 74LS192, U118 7425, U119 74LS151, U12 Conn_02x08_Counter_Clockwise, U120 74LS193, U121 74LS393, U122 74LS145, U123 74LS161, U124 74LS161, U125 74LS161, U126 74LS161, U127 74LS30, U128 74LS161, U129 74LS161, U13 Conn_02x08_Counter_Clockwise, U130 74LS151, U131 74S287, U132 74LS259, U133 74LS107, U134 74LS02, U135 74LS107, U136 74LS74, U137 NE555P, U138 NE555P, U139 74LS02, U14 Conn_02x08_Counter_Clockwise, U140 74LS02, U141 74LS27, U142 74LS00, U143 74LS10, U144 74LS02, U145 74LS27, U146 74LS390, U147 7425, U148 74LS151, U149 Conn_02x08_Counter_Clockwise, U15 Conn_02x08_Counter_Clockwise, U150 74LS145, U151 74LS151, U152 74LS107, U153 74LS10, U154 74LS161, U155 74LS04, U156 74LS10, U157 74LS161, U158 74LS161, U159 74S287, U16 Conn_02x08_Counter_Clockwise, U160 74LS107, U161 74LS153, U162 74LS42, U163 74S287, U164 74LS151, U165 74LS151, U166 74LS161, U167 74LS00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

Commit message: schem
Connections:
- net at U53.2: now also U78.2
- net at U167.10, U72.6: now also U130.6 (~{Z})
- net at U24.14 (Q0): now also U78.1
- net at U186.9: now also U184.9
- net at U100.14 (S0), U101.5: now also U131.10 (Q2)
Other:
- moved on the sheet: U78A
Changed lines of the file:
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@@
 	)
 	(junction
+		(at 750.57 -394.97)
+		(diameter 0)
+		(color 0 0 0 0)
+	)
+	(junction
 		(at 1076.96 -39.37)
 		(diameter 0)
@@
 	)
 	(junction
+		(at 1591.31 -200.66)
+		(diameter 0)
+		(color 0 0 0 0)
+	)
+	(junction
 		(at 1437.64 -379.73)
 		(diameter 0)
@@
 	(wire
 		(pts
+			(xy 624.84 -22.86) (xy 624.84 -394.97)
+		)
+		(stroke
+			(width 0)
+			(type default)
+		)
+	)
+	(wire
+		(pts
 			(xy 782.32 -195.58) (xy 765.81 -195.58)
 		)
@@
 	(wire
 		(pts
+			(xy 624.84 -394.97) (xy 750.57 -394.97)
+		)
+		(stroke
+			(width 0)
+			(type default)
+		)
+	)
+	(wire
+		(pts
 			(xy 1234.44 233.68) (xy 1225.55 233.68)
 		)
@@
 	(wire
 		(pts
+			(xy 861.06 -280.67) (xy 928.37 -280.67)
+		)
+		(stroke
+			(width 0)
+			(type default)
+		)
+	)
+	(wire
+		(pts
 			(xy 487.68 -288.29) (xy 487.68 -280.67)
 		)
@@
 	(wire
 		(pts
+			(xy 1591.31 -491.49) (xy 928.37 -491.49)
+		)
+		(stroke
+			(width 0)
+			(type default)
+		)
+	)
+	(wire
+		(pts
 			(xy 679.45 -44.45) (xy 674.37 -44.45)
 		)
@@
 	(wire
 		(pts
+			(xy 1109.98 951.23) (xy 1109.98 864.87)
+		)
+		(stroke
+			(width 0)
+			(type default)
+		)
+	)
+	(wire
+		(pts
 			(xy 514.35 -293.37) (xy 524.51 -293.37)
 		)
@@
 	(wire
 		(pts
-			(xy 1676.4 544.83) (xy 1676.4 530.86)
+			(xy 1678.94 544.83) (xy 1678.94 530.86)
 		)
 		(stroke
@@
 	(wire
 		(pts
-			(xy 1676.4 530.86) (xy 1616.71 530.86)
+			(xy 1678.94 530.86) (xy 1616.71 530.86)
 		)
 		(stroke
@@
 	(wire
 		(pts
+			(xy 1687.83 537.21) (xy 1671.32 537.21)
+		)
+		(stroke
+			(width 0)
+			(type default)
+		)
+	)
+	(wire
+		(pts
 			(xy 821.69 434.34) (xy 854.71 434.34)
 		)
@@
 	(wire
 		(pts
+			(xy 1112.52 951.23) (xy 1109.98 951.23)
+		)
+		(stroke
+			(width 0)
+			(type default)
+		)
+	)
+	(wire
+		(pts
 			(xy 171.45 623.57) (xy 168.91 623.57)
 		)
@@
 	(wire
 		(pts
-			(xy 1619.25 533.4) (xy 1673.86 533.4)
+			(xy 1619.25 533.4) (xy 1677.67 533.4)
 		)
 		(stroke
@@
 	(wire
 		(pts
+			(xy 1671.32 537.21) (xy 1671.32 544.83)
+		)
+		(stroke
+			(width 0)
+			(type default)
+		)
+	)
+	(wire
+		(pts
 			(xy 1037.59 19.05) (xy 1035.05 19.05)
 		)
@@
 	(wire
 		(pts
-			(xy 1656.08 547.37) (xy 1671.32 547.37)
+			(xy 1656.08 547.37) (xy 1676.4 547.37)
 		)
 		(stroke
@@
 	(wire
 		(pts
+			(xy 1591.31 -200.66) (xy 1591.31 -491.49)
+		)
+		(stroke
+			(width 0)
+			(type default)
+		)
+	)
+	(wire
+		(pts
 			(xy 358.14 532.13) (xy 354.33 532.13)
 		)
@@
 	(wire
 		(pts
+			(xy 765.81 854.71) (xy 765.81 864.87)
+		)
+		(stroke
+			(width 0)
+			(type default)
+		)
+	)
+	(wire
+		(pts
 			(xy 22.86 996.95) (xy 26.67 996.95)
 		)
@@
 	(wire
 		(pts
+			(xy 765.81 864.87) (xy 1109.98 864.87)
+		)
+		(stroke
+			(width 0)
+			(type default)
+		)
+	)
+	(wire
+		(pts
 			(xy 734.06 811.53) (xy 697.23 811.53)
 		)
@@
 	(wire
 		(pts
-			(xy 1673.86 547.37) (xy 1687.83 547.37)
+			(xy 1677.67 547.37) (xy 1687.83 547.37)
 		)
 		(stroke
@@
 	(wire
 		(pts
-			(xy 1671.32 547.37) (xy 1671.32 534.67)
+			(xy 1676.4 547.37) (xy 1676.4 534.67)
 		)
 		(stroke
@@
 	(wire
 		(pts
+			(xy 928.37 -491.49) (xy 928.37 -280.67)
+		)
+		(stroke
+			(width 0)
+			(type default)
+		)
+	)
+	(wire
+		(pts
 			(xy 491.49 -73.66) (xy 491.49 -113.03)
 		)
@@
 	(wire
 		(pts
-			(xy 1671.32 534.67) (xy 1687.83 534.67)
+			(xy 1676.4 534.67) (xy 1687.83 534.67)
 		)
 		(stroke
@@
 	(wire
 		(pts
-			(xy 1687.83 544.83) (xy 1676.4 544.83)
+			(xy 1687.83 544.83) (xy 1678.94 544.83)
 		)
 		(stroke
@@
 	(wire
 		(pts
-			(xy 1673.86 533.4) (xy 1673.86 547.37)
+			(xy 1677.67 533.4) (xy 1677.67 547.37)
 		)
 		(stroke
@@
 	(wire
 		(pts
+			(xy 553.72 -22.86) (xy 624.84 -22.86)
+		)
+		(stroke
+			(width 0)
+			(type default)
+		)
+	)
+	(wire
+		(pts
 			(xy 723.9 834.39) (xy 723.9 824.23)
 		)
@@
 	(text "O"
 		(exclude_from_sim no)
-		(at 579.882 -129.032 0)
+		(at 750.316 -394.97 0)
 		(effects
 			(font
@@
 	(symbol
 		(lib_id "74xx:74LS04")
-		(at 281.94 245.11 0)
+		(at 1663.7 544.83 0)
 		(unit 1)
 		(exclude_from_sim no)
@@
 		(fields_autoplaced yes)
 		(property "Reference" "U78"
-			(at 281.94 236.22 0)
+			(at 1663.7 535.94 0)
 			(effects
 				(font
@@
 		)
 		(property "Value" "74LS04"
-			(at 281.94 238.76 0)
+			(at 1663.7 538.48 0)
 			(effects
 				(font
@@
 		)
 		(property "Footprint" "Package_DIP:DIP-14_W7.62mm"
-			(at 281.94 245.11 0)
+			(at 1663.7 544.83 0)
 			(effects
 				(font
@@
 		)
 		(property "Datasheet" "http://www.ti.com/lit/gpn/sn74LS04"
-			(at 281.94 245.11 0)
+			(at 1663.7 544.83 0)
 			(effects
 				(font
@@
 		)
 		(property "Description" ""
-			(at 281.94 245.11 0)
+			(at 1663.7 544.83 0)
 			(effects
 				(font

Commit message: move closer together
Connections:
- net C37: now also C5.2
- net VCC: no longer U207.6 (A2), U209.11 (S0), U212.12 (Q2), U214.6 (A1), U215.4, U241.4, U31.10 (CET), U94.4
- net at U206.1 (S), U207.23 (A8): now also U118.2; no longer U118.3 (G), U233.6 (~{Z})
- net at U198.13, U199.14 (~{R}), U201.8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: no longer U112.2 (CP), U113.2 (CP)
- net at U63.11: now also U89.4
- net at U54.3 (D0): now also U20.3
- net at U54.4 (D1): now also U20.2
- net at U213.2 (S1): now also U187.5 (A3)
- net at U239.11 (K), U239.13 (~{R}): now also U239.6 (~{Q})
- net at Q1.2 (C): now also D2.2 (A), J1.29 (Pin_29)
- net at U119.10 (S1), U148.10 (S1), U177.10 (S1)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: no longer U117.6 (QC), U118.10, U148.2 (I2)
- net at U165.15 (I4), U194.5 (A0): no longer U165.14 (I5)
- net at U194.6 (A1): now also U165.14 (I5)
- net at U194.9 (Q3): now also U165.12 (I7)
- net at U119.7 (~{E}), U148.7 (~{E}), U177.7 (~{E})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: now also U180.9 (Zb); no longer U117.3 (QA), U118.12, U90.2 (I2)
- net at U104.14 (~{R}), U104.6 (~{S}), U124.10 (CET)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: now also U220.9
- net at U51.6 (A2), U80.12 (Q2): no longer U51.8 (A0), U80.14 (Q0)
- net at U59.5 (Q2), U60.2 (A5), U61.2 (A5): no longer U59.4 (Q1), U60.3 (A4), U61.3 (A4)
- net at U48.9 (S0): now also U26.3 (D0)
- net at U220.5: now also U191.3 (2)
- net at U187.3 (A5): now also U214.3 (A4)
- net at U187.4 (A4): now also U214.4 (A3)
- net at U251.6 (Oa=b): now also U219.4 (2C), U227.12
- net at U199.3 (~{S2}): now also U199.12 (~{S2})
- net at U249.13 (CP): now also U220.13
- new net: U207.6 (A2), U209.11 (S0), U212.12 (Q2), U214.6 (A1), U215.4, U241.4
- new net: U31.10 (CET), U94.4
- new net: U51.8 (A0), U80.14 (Q0)
- new net: U59.4 (Q1), U60.3 (A4), U61.3 (A4)
- new net: U112.2 (CP), U113.2 (CP)
- new net: U117.6 (QC), U118.10, U148.2 (I2)
- new net: U117.3 (QA), U118.12
- now unconnected: U59.10 (Q1), U94.2, U96.3
Other:
- moved on the sheet: C10, C11, C12, C13, C14, C15, C16, C17, C18, C2, C26, C27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

Commit message: add pcb file
Connections:
- net at U152.10 (~{R}), U152.13 (~{R}): now also U153.9
- net at U218.5, U249.12 (MR): now also U226.4
Changed lines of the file:
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@@
 	)
 	(junction
+		(at 356.87 474.98)
+		(diameter 0)
+		(color 0 0 0 0)
+	)
+	(junction
 		(at 497.84 -342.9)
 		(diameter 0)
@@
 	)
 	(junction
+		(at 1209.04 739.14)
+		(diameter 0)
+		(color 0 0 0 0)
+	)
+	(junction
 		(at 1323.34 744.22)
 		(diameter 0)
@@
 	)
 	(junction
-		(at 1082.04 284.48)
-		(diameter 0)
-		(color 0 0 0 0)
-	)
-	(junction
 		(at 1216.66 289.56)
 		(diameter 0)
@@
 	(wire
 		(pts
-			(xy 1082.04 284.48) (xy 1082.04 447.04)
-		)
-		(stroke
-			(width 0)
-			(type default)
-		)
-	)
-	(wire
-		(pts
 			(xy 137.16 -490.22) (xy 116.84 -490.22)
 		)
@@
 	(wire
 		(pts
+			(xy 580.39 -128.27) (xy 580.39 -132.08)
+		)
+		(stroke
+			(width 0)
+			(type default)
+		)
+	)
+	(wire
+		(pts
 			(xy 1314.45 -242.57) (xy 1314.45 -248.92)
 		)
@@
 	(wire
 		(pts
+			(xy 633.73 463.55) (xy 1209.04 463.55)
+		)
+		(stroke
+			(width 0)
+			(type default)
+		)
+	)
+	(wire
+		(pts
 			(xy 656.59 -436.88) (xy 645.16 -436.88)
 		)
@@
 	(wire
 		(pts
+			(xy 633.73 -132.08) (xy 633.73 463.55)
+		)
+		(stroke
+			(width 0)
+			(type default)
+		)
+	)
+	(wire
+		(pts
 			(xy 1630.68 494.03) (xy 1615.44 494.03)
 		)
@@
 	(wire
 		(pts
+			(xy 356.87 534.67) (xy 356.87 474.98)
+		)
+		(stroke
+			(width 0)
+			(type default)
+		)
+	)
+	(wire
+		(pts
 			(xy 933.45 748.03) (xy 933.45 750.57)
 		)
@@
 	(wire
 		(pts
+			(xy 561.34 534.67) (xy 356.87 534.67)
+		)
+		(stroke
+			(width 0)
+			(type default)
+		)
+	)
+	(wire
+		(pts
 			(xy 455.93 -248.92) (xy 455.93 -303.53)
 		)
@@
 	(wire
 		(pts
+			(xy 561.34 525.78) (xy 561.34 534.67)
+		)
+		(stroke
+			(width 0)
+			(type default)
+		)
+	)
+	(wire
+		(pts
 			(xy 1042.67 24.13) (xy 1042.67 -39.37)
 		)
@@
 	(wire
 		(pts
+			(xy 1209.04 463.55) (xy 1209.04 739.14)
+		)
+		(stroke
+			(width 0)
+			(type default)
+		)
+	)
+	(wire
+		(pts
 			(xy 938.53 816.61) (xy 875.03 816.61)
 		)
@@
 	(wire
 		(pts
+			(xy 580.39 -132.08) (xy 633.73 -132.08)
+		)
+		(stroke
+			(width 0)
+			(type default)
+		)
+	)
+	(wire
+		(pts
 			(xy 1234.44 175.26) (xy 1226.82 175.26)
 		)
@@
 	(text "O"
 		(exclude_from_sim no)
-		(at 494.538 500.38 0)
+		(at 1214.374 749.046 0)
 		(effects
 			(font
