File: Main.kicad_sch (KiCad schematic)
At the start: 449 parts, among them J1 Conn_02x22_Top_Bottom, Q1 2SC1384, Q2 2SC1384, SW1 SW_DIP_x08, U1 Conn_02x08_Counter_Clockwise, U10 7416, U100 74LS153, U101 74LS86, U102 74LS151, U103 74LS153, U104 74LS279, U105 74LS00, U106 74LS08, U107 NE555P, U108 74LS161, U109 74LS107, U11 7416, U110 74LS10, U111 74LS157, U112 74LS161, U113 74LS161, U114 74LS107, U115 Conn_02x08_Counter_Clockwise, U116 74LS175, U117 74LS192, U118 7425, U119 74LS151, U12 Conn_02x08_Counter_Clockwise, U120 74LS193, U121 74LS393, U122 74LS145, U123 74LS161, U124 74LS161, U125 74LS161, U126 74LS161, U127 74LS30, U128 74LS161, U129 74LS161, U13 Conn_02x08_Counter_Clockwise, U130 74LS151, U131 74S287, U132 74LS259, U133 74LS107, U134 74LS02, U135 74LS107, U136 74LS74, U137 NE555P, U138 NE555P, U139 74LS02, U14 Conn_02x08_Counter_Clockwise, U140 74LS02, U141 74LS27, U142 74LS00, U143 74LS10, U144 74LS02, U145 74LS27, U146 74LS390, U147 7425, U148 74LS151, U149 Conn_02x08_Counter_Clockwise, U15 Conn_02x08_Counter_Clockwise, U150 74LS145, U151 74LS151, U152 74LS107, U153 74LS10, U154 74LS161, U155 74LS04, U156 74LS10, U157 74LS161, U158 74LS161, U159 74S287, U16 Conn_02x08_Counter_Clockwise, U160 74LS107, U161 74LS153, U162 74LS42, U163 74S287, U164 74LS151, U165 74LS151, U166 74LS161, U167 74LS00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

Commit message: moar
Connections:
- net CLOCK_B: now also U227.10, U227.9
- net at U71.1 (~{R}), U71.8 (~{Q}): now also U68.1 (~{R})
- net UP LEFT: now reaches U46.4 (1Q), U47.11, U48.4 (I7)
- net DOWN LEFT: now reaches U46.9 (3Q), U47.8, U48.11 (I1)
- net CLOCK_D: now reaches U108.2 (CP), U112.2 (CP), U113.2 (CP), U166.2 (CP), U79.2 (CP), U80.2 (CP), U81.2 (CP), U85.2 (CP), U86.2 (CP)
- net CLOCK_D: now also U227.8
- net COIN IN: now reaches U11.1, U41.5, U42.11 (C), U75.7 (Q)
- net at R80.1, U42.1 (~{R}), U42.13 (~{R})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: now also U40.10, U7.4 (~{Q})
- net at U38.4 (R), U40.13: now also C63.2, U145.8
- net UP RIGHT: now reaches U75.4 (Q), U76.11, U77.4 (I7)
- net at U69.1, U70.1: now also C58.2, U178.6 (~{Z})
- net at U70.6: now also C143.1
- net at U221.3 (~{Q0}): now also U243.6
- net at U168.4 (E23), U171.7 (Q1): now also U104.11 (~{S1})
- net at C57.2, R66.1, R67.1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: now also R70.2
- net at U170.9: now also U170.12
- net at U190.5, U226.5, U258.12 (A3): now also U183.11 (Q3)
- net SHOOT LEFT: now reaches U104.4 (Q), U73.4, U78.11
- net DOWN RIGHT: now reaches U75.9 (Q), U76.8, U77.11 (I1)
- net at U106.13, U77.12 (I2): now also U144.8, U170.4, U171.14 (~{Q3}), U51.23 (A8)
- net at U74.3: now also U223.12
- net at U47.9, U76.9: now also U258.11 (9)
- net at U38.3 (Q): now also U74.11
- net at U183.12 (Q2): now also U187.23 (A8)
- net at U83.6 (~{Z}): now also U6.9, U72.1
- net at U257.4 (3): now also U98.10
- net at U73.10, U78.3: now also U117.13 (~{BO}), U68.12 (D), U89.12
- net SHOOT RIGHT: now reaches U104.9 (Q), U73.1, U78.5
- net NEW GAME START: now reaches U42.3 (C), U43.4 (1Q), U73.12
- net at U160.3 (Q), U161.14 (S0): now also U231.14 (S0)
- net at U100.2 (S1), U101.4: now also U131.11 (Q1)
- net at U68.11 (C): now also U74.10
- net AUDIO C renamed SHOOT AUDIO
- net C29 renamed COIN METER POWERON
- no-connect marks 534 -> 541
Other:
- moved on the sheet: H1, H2, H3, H4, U227C, U71B, U74E

Commit message: progress!!!!
Connections:
- net RAM_A0: now also U101.1, U155.5, U184.5, U214.1 (A6), U234.11 (I0c), U234.5 (I0b), U234.6 (I1b), U237.10 (S1), U240.13 (Q1)
- net RAM_A1: now also U101.2, U102.11 (S0), U139.11, U184.9, U186.9, U193.13 (~{G1}), U234.2 (I0a), U234.3 (I1a), U237.11 (S0), U240.14 (Q0), U242.13
- net RAM_A2: now also U100.4 (I2a), U103.2 (S1), U132.2 (A1), U151.9 (S2), U184.10, U214.15 (A7), U215.1, U233.9 (S2), U234.14 (I0d), U237.9 (S2), U240.12 (Q2), U241.5, U242.12, U74.5, U99.11
- net RAM_A3: now also U131.12 (Q0), U183.12 (Q2), U187.23 (A8), U223.11; no longer U143.4
- net RAM_A4: now also U234.10 (I1c), U240.11 (Q3), U241.6
- net RAM_A5: now also U234.13 (I1d), U239.3 (Q), U241.11
- net RAM_A6: now also U100.14 (S0), U101.5, U131.10 (Q2), U155.13, U183.14 (Q0), U187.2 (A6), U215.2
- net RAM_A7: now also U100.2 (S1), U101.4, U131.11 (Q1), U183.13 (Q1), U187.1 (A7)
- net U258_3: now also U243.8
- net at U136.9 (Q), U190.4, U230.1 (~{R})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: now also U180.1 (Ea)
- net at U118.2, U206.1 (S), U207.23 (A8): now also U243.10
- net at U207.5 (A3), U209.10 (S1), U212.11 (Q3)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: now also U191.12 (A3), U193.12 (Q0), U194.13 (~{G1})
- net at U207.7 (A1), U212.13 (Q1), U214.5 (A0)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: now also U191.14 (A1), U192.10 (S1), U193.10 (Q2), U194.11 (Q1)
- net at C59.1, U136.11 (C), U151.1 (I3)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: now also U237.12 (I7), U237.13 (I6), U237.3 (I1)
- net at U131.13 (~{G1}), U151.12 (I7), U151.13 (I6)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: now also U206.13 (I1d), U237.14 (I5), U237.15 (I4), U237.2 (I2)
- net at U151.5 (Z): now also U118.1
- net at U151.7 (~{E}): now also U180.15 (Eb), U233.7 (~{E}), U6.11
- net at U223.5, U225.5, U226.10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: now also U132.13 (D)
- net at C35.1, U221.13 (D3), U226.11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: now also U256.6 (~{DO})
- net at U242.1, U243.1: now also U156.3, U158.3 (D0)
- net at U160.9 (C), U242.2: now also U160.3 (Q), U161.14 (S0), U231.14 (S0)
- net at U140.9, U197.13 (1B): now also U198.1
- net at U71.10 (~{S}): now also U152.10 (~{R}), U152.13 (~{R}), U153.9, U222.2, U239.11 (K), U239.13 (~{R}), U239.6 (~{Q})
- net at U145.10, U46.13 (4Q): now also U65.13 (1B)
- net at U63.12: now also U97.4
- net at U139.8: now also U200.6
- net at U114.3 (Q), U56.3: now also U110.10
- net at U153.1, U182.5 (Q): now also U126.3 (D0), U136.3 (C)
- net at U153.12, U181.1 (CP): now also C36.1, U101.13, U220.11, U243.2, U248.3 (C), U32.4 (DOWN), U41.9
- net at U153.13, U153.4, U154.12 (Q2): now also U39.2
- net at U106.12, U106.2, U11.11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: now also U199.12 (~{S2}), U199.3 (~{S2})
- net at C63.2, U145.8, U38.4 (R)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: now also U137.4 (R), U201.13, U208.4, U225.9
- net at U201.3, U201.4, U202.2 (TR)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: now also U9.9 (A), U93.11 (~{S1})
- net at U70.12: now also U63.6
- net at U70.2: now also U139.4
- net at U70.3: now also U225.8
- net at U69.5, U70.5: now also U225.12, U226.13
- net at C143.1, U70.6: now also U182.2 (~{Q})
- net at U50.8: now also U141.4
- net at U181.10 (Q1): now also U39.8
- net at U181.11 (Q0): now also U40.1
- net at U181.13 (CP), U181.6 (Q3): now also U165.7 (~{E}), U244.12 (C)
- net at U218.3, U221.2 (Q0): now also U225.2
- net at U218.4, U221.7 (Q1): now also U247.1 (~{MR})
- net at U169.5 (~{R}), U198.3: now also U198.12
- net at U220.2: now also U191.5 (4)
- net at U220.3: now also U162.6 (5)
- net at U153.3, U154.14 (Q0): now also U213.14 (S0)
- net at U213.1 (Ea): now also U105.6
- net at U213.7 (Za): now also U210.5, U69.4
- net at U239.2 (~{Q}), U242.5: now also U136.12 (D)
- net at U128.9 (~{PE}), U129.9 (~{PE}): now also U98.6
- net at U127.4: now also U158.11 (Q3)
- net at U234.1 (S): now also U155.4, U180.4 (I2a), U180.5 (I1a)
- net at U167.9, U197.6 (2Y): now also U72.5
- net at U245.1 (Ea): now also U222.11, U223.13, U225.1, U230.12 (D), U230.13 (~{R})
- net at C62.1, U135.12 (C), U135.9 (C)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: now also U181.3 (Q0)
- net at U108.13 (Q1): now also U111.5 (I0b)
- net at U108.15 (TC), U79.7 (CEP): now also U110.1
- net at C64.2, U142.6, U84.7 (~{E}): now also U111.1 (S)
- net at U193.11 (Q1), U194.12 (Q0): now also U191.13 (A2), U192.9 (S2)
- net at U156.9, U162.12 (A3), U163.13 (~{G1})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: now also U134.2, U178.9 (S2), U187.3 (A5), U214.3 (A4)
- net at U123.1 (~{MR}), U124.1 (~{MR}), U125.1 (~{MR})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: now also U211.13 (~{R})
- net at U244.3 (Q): now also U156.4, U8.10 (B)
- net at U90.12 (I7): now also U175.3 (Q0), U175.4 (~{CP1}), U176.1, U205.9
- net at U90.13 (I6): now also U120.3 (QA)
- net at U90.14 (I5): now also U146.12 (~{CP1}), U146.13 (Q0), U147.13, U150.15 (P0), U205.4
- net at U175.12 (~{CP1}), U175.13 (Q0), U176.13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: now also U179.15 (P0)
- net at U104.14 (~{R}), U104.6 (~{S}), U124.10 (CET)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: now also U182.11 (K), U182.13 (~{R}), U182.6 (~{Q})
- net at U125.9 (~{PE}), U126.9 (~{PE}), U92.4: now also U93.3 (~{S2}), U97.8
- net at U92.11: now also U106.9
- net at U92.13: now also R58.1, U37.1 (Q0), U37.9 (Q7)
- net at U104.13 (Q): now also U246.10, U246.13, U246.4
- net at U75.15 (~{S}): now also U190.8
- net at U59.10 (Q1): now also U94.13, U96.2
- net at U59.12 (MR), U59.2 (MR): now also U94.2
- net at U49.9: now also U171.5 (D1), U199.9 (Q), U200.1
- net at U137.3 (Q), U196.11, U200.9: now also U244.8 (J)
- net at U116.12 (D2), U116.7 (Q1): now also U199.11 (~{S1})
- net at U33.12 (MR), U33.2 (MR): now also U94.10, U96.11
- net at U89.5: now also U91.13 (~{BO}), U92.1
- net at U89.2, U92.2: now also U120.13 (~{BO}), U65.9 (1C)
- net at U88.11 (~{LOAD}): now also U117.11 (~{LOAD}), U42.6 (~{Q}), U73.13
- net at U88.2 (QB): now also U119.3 (I1)
- net at U88.7 (QD): now also U177.3 (I1)
- net at U233.2 (I2): now also U118.8
- net at U233.6 (~{Z}): now also U118.3 (G)
- net at U198.11: now also U169.1 (~{R}), U169.10 (~{R})
- net at U98.12, U99.3: now also U129.5 (D2), U161.9 (Zb)
- net at U98.13: now also U244.11 (K), U244.5 (Q)
- net at U211.12 (C): now also U125.15 (TC), U97.10
- net at U211.3 (Q): now also U97.11
- net at U152.1 (J), U152.4 (K), U152.5 (Q): now also U180.12 (I2b), U206.10 (I1c)
- net at U152.12 (C), U152.9 (C), U155.6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: now also U102.10 (S1)
- net at U183.15 (TC): now also U182.1 (J)
- net at C70.1, U121.2 (MR): now also U8.2 (B)
- net at U215.8, U216.9 (S2): now also U185.11 (S0)
- net at U155.3: now also U257.4 (3), U98.10
- net at U201.5, U202.3 (Q): now also U255.13 (DI)
- net at U102.6 (~{Z}): now also U243.5
- net at U102.9 (S2): now also U186.12, U186.2
- net at U181.4 (Q1): now also U36.1 (CP), U64.1
- net at U181.5 (Q2): now also U64.13
- net at U208.8: now also U34.11 (~{LOAD})
- net at U175.10 (Q2), U176.10: now also U148.4 (I0), U179.13 (P2)
- net at U175.11 (Q1), U176.12: now also U119.4 (I0), U179.14 (P1)
- net at U175.9 (Q3), U176.9, U177.4 (I0)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: now also U179.12 (P3)
- net at U101.3: now also U105.1
- net at U219.10 (1D), U219.3 (2B): now also U105.11
- net at U229.10: now also U192.7 (~{E})
- net at U146.1 (~{CP0}): now also U204.6
- net at U146.5 (Q1), U147.2: now also U119.15 (I4)
- net at U146.15 (~{CP0}), U146.7 (Q3), U147.5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: now also U177.15 (I4)
- net at U257.9 (7): now also U243.11
- net at U119.12 (I7): now also U175.5 (Q1), U176.2
- net at U119.13 (I6): now also U120.2 (QB)
- net at U97.3: now also U226.3, U229.12, U249.5 (Q2)
- net at U97.5: now also U63.1
- net at U97.6: now also U7.10 (B)
- net at U109.9 (C), U110.13: now also U79.15 (TC)
- net at U175.6 (Q2), U176.4: now also U148.12 (I7)
- net at U21.13 (Q1): now also U84.10 (S1)
- net at U21.14 (Q0): now also U84.11 (S0)
- net at U143.8: now also U225.11
- net at U223.10: now also U186.3
- net at U223.8: now also U105.2
- net at U255.12 (~{WE}): now also U201.6
- net at U224.10, U224.4: now also U192.5 (Z)
- net at U171.4 (D0), U199.4 (Q), U200.3: now also U49.13
- net at U141.3: now also U22.14 (Q0)
- net at U134.8: now also U161.7 (Za)
- net at U182.10 (~{R}): now also U155.12
- net at U187.4 (A4), U214.4 (A3): now also U178.10 (S1)
- net at U206.11 (I0c): now also U148.5 (Z)
- net at U225.10: now also U105.9
- net at U146.10 (Q2), U147.10, U148.14 (I5): now also U150.13 (P2)
- net at U146.9 (Q3), U147.9: now also U150.12 (P3), U177.14 (I5), U205.5
- net at U89.3: now also U120.4 (DOWN)
- net at U105.13: now also U135.6 (~{Q})
- net at U231.3 (I3a), U259.3 (2): now also U199.15 (~{S})
- net at U199.1 (~{R}): now also U49.5, U73.6
- net at U152.6 (~{Q}): now also U180.13 (I3b)
- net at U180.7 (Za): now also U118.4, U118.5
- net at U64.12, U64.2: now also U34.12 (~{CO})
- net at U162.13 (A2), U163.12 (Q0): now also U164.9 (S2), U165.9 (S2)
- net at U148.13 (I6): now also U120.6 (QC)
- net at U117.7 (QD), U118.9: now also U177.2 (I2)
- net at U120.7 (QD): now also U177.13 (I6)
- net at U49.4, U73.3: now also U199.10 (~{R})
- net at U185.6 (~{Z}): now also U72.4
- net at U93.13 (Q), U94.1: now also U30.1 (~{MR})
- net at U178.7 (~{E}): now also U118.6
- net at U227.2: now also U191.10 (8)
- new net U25X_A2: U143.4
- no-connect marks 541 -> 593
Other:
- moved on the sheet: C52, C53, R75, R76, U101A, U10D, U10E, U114A, U120, U139C, U155F, U193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

Commit message: NC
Connections:
- net RAM_A7: now also U74.9
- net at U39.13, U41.2: now also U74.13
- net at U71.9 (Q): now also U153.11
- net at U63.12, U97.4: now also U106.1, U144.12, U170.1, U171.11 (~{Q2}), U48.12 (I2), U57.23 (A8)
- net U258_7: now reaches U139.9, U143.11, U258.7 (6)
- net at U169.5 (~{R}), U198.3: no longer U198.12
- net at U152.1 (J), U152.4 (K), U152.5 (Q)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: now also U102.9 (S2), U186.12, U186.2
- net at U121.5 (Q2), U122.13 (P2): now also U131.14 (~{G2})
- net at U136.8 (~{Q}): now also U243.12, U243.9
- net at U145.11: now also U236.6 (~{Q})
- net U258_9: now reaches U139.12
- net U258_9: now also U143.10, U258.9 (7)
- net at U43.5 (*2R): now also U74.12
- net U258_5: now reaches U258.5 (4)
- net U258_6: now reaches U258.6 (5)
- net U258_6: now also U198.12
- no-connect marks 593 -> 605
Other:
- moved on the sheet: U74F
