File: Main.kicad_sch (KiCad schematic)
At the start: 449 parts, among them J1 Conn_02x22_Top_Bottom, Q1 2SC1384, Q2 2SC1384, SW1 SW_DIP_x08, U1 Conn_02x08_Counter_Clockwise, U10 7416, U100 74LS153, U101 74LS86, U102 74LS151, U103 74LS153, U104 74LS279, U105 74LS00, U106 74LS08, U107 NE555P, U108 74LS161, U109 74LS107, U11 7416, U110 74LS10, U111 74LS157, U112 74LS161, U113 74LS161, U114 74LS107, U115 Conn_02x08_Counter_Clockwise, U116 74LS175, U117 74LS192, U118 7425, U119 74LS151, U12 Conn_02x08_Counter_Clockwise, U120 74LS193, U121 74LS393, U122 74LS145, U123 74LS161, U124 74LS161, U125 74LS161, U126 74LS161, U127 74LS30, U128 74LS161, U129 74LS161, U13 Conn_02x08_Counter_Clockwise, U130 74LS151, U131 74S287, U132 74LS259, U133 74LS107, U134 74LS02, U135 74LS107, U136 74LS74, U137 NE555P, U138 NE555P, U139 74LS02, U14 Conn_02x08_Counter_Clockwise, U140 74LS02, U141 74LS27, U142 74LS00, U143 74LS10, U144 74LS02, U145 74LS27, U146 74LS390, U147 7425, U148 74LS151, U149 Conn_02x08_Counter_Clockwise, U15 Conn_02x08_Counter_Clockwise, U150 74LS145, U151 74LS151, U152 74LS107, U153 74LS10, U154 74LS161, U155 74LS04, U156 74LS10, U157 74LS161, U158 74LS161, U159 74S287, U16 Conn_02x08_Counter_Clockwise, U160 74LS107, U161 74LS153, U162 74LS42, U163 74S287, U164 74LS151, U165 74LS151, U166 74LS161, U167 74LS00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

Commit message: update pcb
Connections:
- net U25X_A2 is gone; now on net RAM_A3: U143.4
- net GND: now also U91.9 (D)
- net VCC: now also U24.10 (CET)
- net at U207.8 (A0): now also U191.15 (A0), U192.11 (S0), U194.10 (Q2), U212.14 (Q0), U230.11 (C), U241.2
- net at U108.3 (D0), U140.3, U167.1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: now also U112.3 (D0), U86.3 (D0)
- net at U46.14 (*4R), U46.5 (*2R): now also U105.13, U135.6 (~{Q})
- net at U145.9, U46.7 (2Q): now also U65.3 (2B)
- net at U210.3: now also U245.7 (Za)
- net at U153.3, U154.14 (Q0), U213.14 (S0): now also U162.15 (A0), U163.10 (Q2), U164.11 (S0), U165.11 (S0), U178.11 (S0), U49.1
- net at U187.5 (A3), U213.2 (S1): now also U162.14 (A1), U163.11 (Q1), U164.10 (S1), U165.10 (S1), U49.2
- net at U183.11 (Q3), U190.5, U226.5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: now also U143.5
- net at U108.14 (Q0): now also U111.2 (I0a)
- net at U134.2, U156.9, U162.12 (A3)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: now also U154.11 (Q3), U155.1
- net at U90.2 (I2): now also U117.3 (QA), U118.12
- net at U106.13, U144.8, U170.4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: now also U63.1, U97.5
- net at U89.5, U91.13 (~{BO}), U92.1: now also U65.4 (2C)
- net at U117.11 (~{LOAD}), U42.6 (~{Q}), U73.13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: now also U201.12
- net at U92.9: now also U231.6 (I0a), U259.4 (3)
- net at U102.10 (S1), U152.12 (C), U152.9 (C)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: now also U242.4
- net at U184.4, U239.5 (Q): now also U143.3
- net at U181.5 (Q2), U64.13: now also U229.11
- net at U101.12, U201.10, U201.9: now also U184.6
- net at U119.2 (I2): now also U117.2 (QB), U118.13
- net at U208.12: now also U162.2 (1)
- net at U208.13: now also U162.1 (0), U220.6
- net at U242.6: now also U185.9 (S2)
- net at U186.8, U187.8 (A0): now also U185.10 (S1)
- net at U36.2 (MR), U68.10 (~{S}): now also U236.5 (Q)
- net at U140.6, U145.2, U145.3: now also U11.3
- net at U110.6: now also U80.9 (~{PE}), U81.9 (~{PE}), U87.1
- net at U89.13: now also U68.11 (C), U74.10
- net at C60.1, U249.1 (CP): now also U229.13
- net at U178.10 (S1), U187.4 (A4), U214.4 (A3): now also U162.13 (A2), U163.12 (Q0), U164.9 (S2), U165.9 (S2)
- net at U39.10: now also U121.13 (CP)
- no-connect marks 605 -> 623
Other:
- moved on the sheet: U11B

Commit message: FINISH
Parts:
- removed U12, U13, U14, U149, U15, U16, U17, U18, U19, U238, U44, U45, U66, U67: Conn_02x08_Counter_Clockwise, symbol Connector_Generic:Conn_02x08_Counter_Clockwise
- removed U20: 74LS07, Package_DIP:DIP-14_W7.62mm, symbol 74xx:74LS07
- added TP1, TP2, TP3, TP4, TP5, TP6: TestPoint, TestPoint:TestPoint_THTPad_D1.5mm_Drill0.7mm, symbol Connector:TestPoint
- added U20: 74LS107, Package_DIP:DIP-14_W7.62mm, symbol 74xx:74LS107
Connections:
- net GND: now also TP1.1, TP2.1, TP3.1, U20.7 (GND)
- net U258_3: now also C61.1, U169.15 (~{S})
- net U258_5: now also U47.12, U76.12
- net VCC: now also U68.13 (~{R}), TP4.1, TP6.1, U20.14 (VCC)
- net at U207.6 (A2), U209.11 (S0), U212.12 (Q2)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: now also U191.13 (A2), U192.9 (S2), U193.11 (Q1), U194.12 (Q0)
- net at U116.9 (Cp), U171.9 (Cp), U21.10 (CET)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: now also U104.14 (~{R}), U104.6 (~{S}), U124.10 (CET), U129.10 (CET), U153.10, U182.11 (K), U182.13 (~{R}), U182.6 (~{Q}), U188.10 (CET), U220.9, U93.14 (~{R}), U95.3 (C)
- net at U23.4 (D1), U77.7 (S1): now also U20.8 (J)
- net at U23.5 (D2), U78.8: now also U20.11 (K)
- net at U140.9, U197.13 (1B), U198.1: now also C64.2, U111.1 (S), U142.6, U84.7 (~{E})
- net at U105.13, U135.6 (~{Q}), U46.14 (*4R)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: now also U120.11 (~{LOAD}), U236.10 (~{S}), U236.4 (~{S}), U91.11 (~{LOAD})
- net at U114.10 (~{R}), U140.10, U85.1 (~{MR})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: now also U26.1 (~{MR}), U27.1 (~{MR})
- net at U86.9 (~{PE}), U87.4: now also U143.12, U85.9 (~{PE})
- net at U153.13, U153.4, U154.12 (Q2)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: now also U162.13 (A2), U163.12 (Q0), U164.9 (S2), U165.9 (S2), U178.10 (S1), U187.4 (A4), U214.4 (A3)
- net at U153.3, U154.14 (Q0), U162.15 (A0)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: no longer U178.11 (S0)
- net at C42.2, R56.2, U7.1 (A): now also TP5.1
- net at U54.3 (D0): now also U20.3 (Q)
- net at U54.4 (D1): now also U20.2 (~{Q})
- net at U162.14 (A1), U163.11 (Q1), U164.10 (S1)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: now also U154.13 (Q1), U178.11 (S0)
- net at U170.12, U170.9: now also U181.4 (Q1), U36.1 (CP), U64.1
- net at U128.1 (~{MR}), U129.1 (~{MR}), U157.1 (~{MR})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: now also U133.10 (~{R}), U134.9, U75.13 (Q)
- net at U128.2 (CP), U129.2 (CP): now also U101.12, U123.2 (CP), U124.2 (CP), U184.6, U201.10, U201.9, U30.2 (CP), U92.5, U93.1 (~{R})
- net at U123.1 (~{MR}), U124.1 (~{MR}), U125.1 (~{MR})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: now also U97.2
- net at U244.10 (~{R}), U244.13 (~{R}): now also U136.6 (~{Q}), U75.14 (~{R})
- net at U125.9 (~{PE}), U126.9 (~{PE}), U92.4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: now also U93.2 (~{S1})
- net at U49.8: now also U20.10 (~{R})
- net at U26.5 (D2), U78.12: now also U20.4 (K)
- net at U59.12 (MR), U59.2 (MR), U94.2: now also U96.3
- net at U21.3 (D0): now also U20.5 (Q)
- net at U21.4 (D1): now also U20.6 (~{Q})
- net at U123.9 (~{PE}), U124.9 (~{PE}): now also U93.15 (~{S}), U98.3
- net at U41.13, U43.6 (*2S): now also U106.10
- net at U219.1 (1A), U220.4: now also U105.9, U225.10
- net at U219.13 (1B): now also U227.11
- net at U6.12: now also U136.8 (~{Q}), U243.12, U243.9
- net at U26.4 (D1), U48.7 (S1): now also U20.1 (J)
- net at U189.9 (~{PE}), U190.11: now also U188.9 (~{PE})
- net at U29.10, U87.11: now also U20.9 (C)
- net at U140.5, U169.12 (~{S2}), U169.2 (~{S1})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: now also U7.11 (Clr), U8.11 (Clr), U9.3 (Clr)
- net at U29.12, U87.8: now also U20.12 (C)
- net at U49.11: now also U20.13 (~{R})
- net at U64.3, U65.2 (2A): now also U39.5, U65.1 (1A)
- no-connect marks 623 -> 421
Other:
- moved on the sheet: U115, U134C

Commit message: fix rest of the warnings
Parts:
- C33: footprint Capacitor_THT:CP_Radial_Tantal_D4.5mm_P5.00mm -> Capacitor_THT:C_Disc_D4.3mm_W1.9mm_P5.00mm
- C49, Cf1, Cf10, Cf11, Cf12, Cf13, Cf14, Cf15, Cf16, Cf17, Cf18, Cf19, Cf2, Cf20, Cf21, Cf22, Cf23, Cf24, Cf25, Cf26, Cf27, Cf28, Cf3, Cf4, Cf40, Cf5, Cf6, Cf7, Cf8, Cf9: footprint Capacitor_THT:C_Disc_D7.5mm_W5.0mm_P10.00mm -> Capacitor_THT:C_Axial_L3.8mm_D2.6mm_P10.00mm_Horizontal
Changed lines of the file:
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@@
 			)
 		)
-		(property "Footprint" "Capacitor_THT:C_Disc_D7.5mm_W5.0mm_P10.00mm"
+		(property "Footprint" "Capacitor_THT:C_Axial_L3.8mm_D2.6mm_P10.00mm_Horizontal"
 			(at -171.1452 248.92 0)
 			(effects
@@
 			)
 		)
-		(property "Footprint" "Capacitor_THT:C_Disc_D7.5mm_W5.0mm_P10.00mm"
+		(property "Footprint" "Capacitor_THT:C_Axial_L3.8mm_D2.6mm_P10.00mm_Horizontal"
 			(at -171.1452 248.92 0)
 			(effects
@@
 			)
 		)
-		(property "Footprint" "Capacitor_THT:C_Disc_D7.5mm_W5.0mm_P10.00mm"
+		(property "Footprint" "Capacitor_THT:C_Axial_L3.8mm_D2.6mm_P10.00mm_Horizontal"
 			(at -171.1452 248.92 0)
 			(effects
@@
 			)
 		)
-		(property "Footprint" "Capacitor_THT:C_Disc_D7.5mm_W5.0mm_P10.00mm"
+		(property "Footprint" "Capacitor_THT:C_Axial_L3.8mm_D2.6mm_P10.00mm_Horizontal"
 			(at -171.1452 248.92 0)
 			(effects
@@
 			)
 		)
-		(property "Footprint" "Capacitor_THT:C_Disc_D7.5mm_W5.0mm_P10.00mm"
+		(property "Footprint" "Capacitor_THT:C_Axial_L3.8mm_D2.6mm_P10.00mm_Horizontal"
 			(at -171.1452 248.92 0)
 			(effects
@@
 			)
 		)
-		(property "Footprint" "Capacitor_THT:C_Disc_D7.5mm_W5.0mm_P10.00mm"
+		(property "Footprint" "Capacitor_THT:C_Axial_L3.8mm_D2.6mm_P10.00mm_Horizontal"
 			(at -171.1452 248.92 0)
 			(effects
@@
 			)
 		)
-		(property "Footprint" "Capacitor_THT:C_Disc_D7.5mm_W5.0mm_P10.00mm"
+		(property "Footprint" "Capacitor_THT:C_Axial_L3.8mm_D2.6mm_P10.00mm_Horizontal"
 			(at -171.1452 248.92 0)
 			(effects
@@
 			)
 		)
-		(property "Footprint" "Capacitor_THT:C_Disc_D7.5mm_W5.0mm_P10.00mm"
+		(property "Footprint" "Capacitor_THT:C_Axial_L3.8mm_D2.6mm_P10.00mm_Horizontal"
 			(at -171.1452 248.92 0)
 			(effects
@@
 			)
 		)
-		(property "Footprint" "Capacitor_THT:C_Disc_D7.5mm_W5.0mm_P10.00mm"
+		(property "Footprint" "Capacitor_THT:C_Axial_L3.8mm_D2.6mm_P10.00mm_Horizontal"
 			(at -171.1452 248.92 0)
 			(effects
@@
 			)
 		)
-		(property "Footprint" "Capacitor_THT:C_Disc_D7.5mm_W5.0mm_P10.00mm"
+		(property "Footprint" "Capacitor_THT:C_Axial_L3.8mm_D2.6mm_P10.00mm_Horizontal"
 			(at -171.1452 248.92 0)
 			(effects
@@
 			)
 		)
-		(property "Footprint" "Capacitor_THT:C_Disc_D7.5mm_W5.0mm_P10.00mm"
+		(property "Footprint" "Capacitor_THT:C_Axial_L3.8mm_D2.6mm_P10.00mm_Horizontal"
 			(at -171.1452 248.92 0)
 			(effects
@@
 			)
 		)
-		(property "Footprint" "Capacitor_THT:C_Disc_D7.5mm_W5.0mm_P10.00mm"
+		(property "Footprint" "Capacitor_THT:C_Axial_L3.8mm_D2.6mm_P10.00mm_Horizontal"
 			(at -171.1452 248.92 0)
 			(effects
@@
 			)
 		)
-		(property "Footprint" "Capacitor_THT:C_Disc_D7.5mm_W5.0mm_P10.00mm"
+		(property "Footprint" "Capacitor_THT:C_Axial_L3.8mm_D2.6mm_P10.00mm_Horizontal"
 			(at -171.1452 248.92 0)
 			(effects
@@
 			)
 		)
-		(property "Footprint" "Capacitor_THT:C_Disc_D7.5mm_W5.0mm_P10.00mm"
+		(property "Footprint" "Capacitor_THT:C_Axial_L3.8mm_D2.6mm_P10.00mm_Horizontal"
 			(at -171.1452 248.92 0)
 			(effects
@@
 			)
 		)
-		(property "Footprint" "Capacitor_THT:C_Disc_D7.5mm_W5.0mm_P10.00mm"
+		(property "Footprint" "Capacitor_THT:C_Axial_L3.8mm_D2.6mm_P10.00mm_Horizontal"
 			(at -171.1452 248.92 0)
 			(effects
@@
 			)
 		)
-		(property "Footprint" "Capacitor_THT:C_Disc_D7.5mm_W5.0mm_P10.00mm"
+		(property "Footprint" "Capacitor_THT:C_Axial_L3.8mm_D2.6mm_P10.00mm_Horizontal"
 			(at -171.1452 248.92 0)
 			(effects
@@
 			)
 		)
-		(property "Footprint" "Capacitor_THT:C_Disc_D7.5mm_W5.0mm_P10.00mm"
+		(property "Footprint" "Capacitor_THT:C_Axial_L3.8mm_D2.6mm_P10.00mm_Horizontal"
 			(at -171.1452 248.92 0)
 			(effects
@@
 			)
 		)
-		(property "Footprint" "Capacitor_THT:C_Disc_D7.5mm_W5.0mm_P10.00mm"
+		(property "Footprint" "Capacitor_THT:C_Axial_L3.8mm_D2.6mm_P10.00mm_Horizontal"
 			(at -171.1452 248.92 0)
 			(effects
@@
 			)
 		)
-		(property "Footprint" "Capacitor_THT:C_Disc_D7.5mm_W5.0mm_P10.00mm"
+		(property "Footprint" "Capacitor_THT:C_Axial_L3.8mm_D2.6mm_P10.00mm_Horizontal"
 			(at -171.1452 248.92 0)
 			(effects
@@
 			)
 		)
-		(property "Footprint" "Capacitor_THT:C_Disc_D7.5mm_W5.0mm_P10.00mm"
+		(property "Footprint" "Capacitor_THT:C_Axial_L3.8mm_D2.6mm_P10.00mm_Horizontal"
 			(at -171.1452 248.92 0)
 			(effects
@@
 			)
 		)
-		(property "Footprint" "Capacitor_THT:C_Disc_D7.5mm_W5.0mm_P10.00mm"
+		(property "Footprint" "Capacitor_THT:C_Axial_L3.8mm_D2.6mm_P10.00mm_Horizontal"
 			(at -171.1452 248.92 0)
 			(effects
@@
 			)
 		)
-		(property "Footprint" "Capacitor_THT:C_Disc_D7.5mm_W5.0mm_P10.00mm"
+		(property "Footprint" "Capacitor_THT:C_Axial_L3.8mm_D2.6mm_P10.00mm_Horizontal"
 			(at -171.1452 248.92 0)
 			(effects
@@
 			)
 		)
-		(property "Footprint" "Capacitor_THT:C_Disc_D7.5mm_W5.0mm_P10.00mm"
+		(property "Footprint" "Capacitor_THT:C_Axial_L3.8mm_D2.6mm_P10.00mm_Horizontal"
 			(at -171.1452 248.92 0)
 			(effects
@@
 			)
 		)
-		(property "Footprint" "Capacitor_THT:CP_Radial_Tantal_D4.5mm_P5.00mm"
+		(property "Footprint" "Capacitor_THT:C_Disc_D4.3mm_W1.9mm_P5.00mm"
 			(at 1341.12 -124.7648 0)
 			(effects
@@
 			)
 		)
-		(property "Footprint" "Capacitor_THT:C_Disc_D7.5mm_W5.0mm_P10.00mm"
+		(property "Footprint" "Capacitor_THT:C_Axial_L3.8mm_D2.6mm_P10.00mm_Horizontal"
 			(at -171.1452 248.92 0)
 			(effects
@@
 			)
 		)
-		(property "Footprint" "Capacitor_THT:C_Disc_D7.5mm_W5.0mm_P10.00mm"
+		(property "Footprint" "Capacitor_THT:C_Axial_L3.8mm_D2.6mm_P10.00mm_Horizontal"
 			(at -171.1452 248.92 0)
 			(effects
@@
 			)
 		)
-		(property "Footprint" "Capacitor_THT:C_Disc_D7.5mm_W5.0mm_P10.00mm"
+		(property "Footprint" "Capacitor_THT:C_Axial_L3.8mm_D2.6mm_P10.00mm_Horizontal"
 			(at -171.1452 248.92 0)
 			(effects
@@
 			)
 		)
-		(property "Footprint" "Capacitor_THT:C_Disc_D7.5mm_W5.0mm_P10.00mm"
+		(property "Footprint" "Capacitor_THT:C_Axial_L3.8mm_D2.6mm_P10.00mm_Horizontal"
 			(at -171.1452 248.92 0)
 			(effects
@@
 			)
 		)
-		(property "Footprint" "Capacitor_THT:C_Disc_D7.5mm_W5.0mm_P10.00mm"
+		(property "Footprint" "Capacitor_THT:C_Axial_L3.8mm_D2.6mm_P10.00mm_Horizontal"
 			(at -171.1452 248.92 0)
 			(effects
@@
 			)
 		)
-		(property "Footprint" "Capacitor_THT:C_Disc_D7.5mm_W5.0mm_P10.00mm"
+		(property "Footprint" "Capacitor_THT:C_Axial_L3.8mm_D2.6mm_P10.00mm_Horizontal"
 			(at -90.17 -304.4952 0)
 			(effects
@@
 			)
 		)
-		(property "Footprint" "Capacitor_THT:C_Disc_D7.5mm_W5.0mm_P10.00mm"
+		(property "Footprint" "Capacitor_THT:C_Axial_L3.8mm_D2.6mm_P10.00mm_Horizontal"
 			(at -171.1452 248.92 0)
 			(effects
